File: electronique/balise émettrice/balise émettrice analogique.brd (EAGLE design)
At the start: 160 x 100 mm, 47 parts, among them IC1 TL084P, IC2 TL084P

Commit message: maj elec balise emettrice
Parts:
- added D6: 1N4004, diode:DO41-10
- added J1: J7MM, jumper:07
- added JP1: (no value), pinhead:1X02
- added S1: (no value), switch:255SB
- added SL1, SL5: (no value), con-amp-quick:07P
- C5, C6, C7, C8: value (none) -> 100n
- D1, D2, D3, D4: value 1N4148DO35-7 -> (none); device diode:DO35-7 -> diode:D-2.5
- R1, R10, R17, R18, R19, R20, R21, R22, R25, R26, R3, R4, R5, R6, R7, R8, R9: device resistor:0204/7 -> resistor:0207/2V
- moved C7 225.0 mm to (57.1, 54.6), turned to 90 degrees
- moved C8 223.4 mm to (62.2, 44.5), turned to 90 degrees
- moved C5 199.4 mm to (31.8, 49.5), turned to 270 degrees
- moved C6 197.1 mm to (31.8, 41.9), turned to 90 degrees
- moved R26 194.6 mm to (2.54, 8.89), turned to 180 degrees
- moved R20 193.8 mm to (68.6, 62.2)
- moved R22 192.7 mm to (55.9, 62.2), turned to 270 degrees
- moved R21 190.6 mm to (59.7, 61.0), turned to 90 degrees
- moved LED2 189.2 mm to (24.1, 1.27), turned to 90 degrees
- moved R19 187.7 mm to (63.5, 62.2)
- moved R18 187.5 mm to (71.1, 59.7), turned to 180 degrees
- moved R25 185.8 mm to (12.7, 7.62), turned to 90 degrees
- moved R17 182.7 mm to (71.1, 57.1)
- moved R23 178.5 mm to (57.1, 14.0), turned to 180 degrees
- moved T1 177.8 mm to (16.5, 6.35), turned to 270 degrees
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Connections:
- new net N$20: D6.A, JP1.1
- new net N$23: D6.C, S1.2
- new net N$25: J1.2, R15.3, R16.3
- net +9V: now also S1.3
- net 0V: now also JP1.2
- net GND: now also SL1.1, SL5.1
- net OUT_1: now also SL1.6, SL5.6
- net OUT_2: now also SL1.7, SL5.7
- net OUT_3: now also SL1.2, SL5.2
- net OUT_4: now also SL1.3, SL5.3
- net OUT_5: now also SL1.4, SL5.4
- net OUT_6: now also SL1.5, SL5.5
- net SIGNAL: now also J1.1; no longer R15.3, R16.3
Routing:
- net SIGNAL: track 0.00 -> 109.3 mm
- net +15V: track 0.00 -> 108.3 mm
- net OUT_3: track 0.00 -> 99.6 mm
- net -15V: track 0.00 -> 99.5 mm
- net 0V: track 0.00 -> 72.8 mm
- net +9V: track 0.00 -> 66.1 mm
- net OUT_4: track 0.00 -> 53.0 mm
- net 40-80HZ: track 0.00 -> 47.4 mm
- net OUT_5: track 0.00 -> 40.7 mm
- net OUT_2: track 0.00 -> 35.2 mm
- net OUT_1: track 0.00 -> 33.7 mm
- net 40KHZ: track 0.00 -> 29.8 mm
- net N$10: track 0.00 -> 29.8 mm
- net N$22: track 0.00 -> 25.7 mm
- net OUT_6: track 0.00 -> 24.7 mm
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- added copper zone on layer 16, net 0V
- added copper zone on layer 16, net GND
Other:
- board size 160 x 100 mm -> 74.9 x 74.9 mm
