File: electronique/balise réceptrice/balise réceptrice - partie filtrage.brd (EAGLE design)
At the start: 160 x 100 mm, 35 parts, among them IC1 TL084P, IC2 TL084P, IC3 TL084P

Commit message: maj filtrage + ajout routage balise receptrice, partie filtrage
Parts:
- added C13, C14, C16: 47n, resistor:C050-024X044
- added C15: 2n2, resistor:C050-024X044
- added C17, C18, C19, C20, C21, C22: 100n, resistor:C050-024X044
- added INPUT: (no value), pinhead:1X02
- added JP2, JP3: (no value), pinhead:1X01
- added R19, R20, R25: 100K, resistor:RTRIM3339P
- added R21: 82K, resistor:0207/2V
- added R22: 150K, resistor:0207/2V
- added R23, R24: 180K, resistor:0207/2V
- added R26, R27: 2K2, resistor:0207/2V
- added SL1: (no value), con-amp-quick:09P
- added U$2, U$3: RJ45_FEMELLE, libINTech-Balise:RJ45_FEMELLE
- added U$4: SWITCH_DP3T_SP112, libINTech-Balise:SWITCH_SP112
- JP1: device pinhead:1X08 -> pinhead:1X01
- R1, R12, R15, R18, R2, R4: device resistor:0204/7 -> resistor:0207/2V
- R11: value 82K -> 47K; device resistor:0204/7 -> resistor:0207/2V
- R13, R16: value 220 -> 1K8; device resistor:0204/7 -> resistor:0207/2V
- R14, R17: value 1K -> 2K
- R3: value 560 -> 470; device resistor:0204/7 -> resistor:0207/2V
- R9: value 82K -> 47K
- moved U$1 224.1 mm to (35.6, 62.2), turned to 90 degrees
- moved C11 195.3 mm to (58.4, 27.9)
- moved R16 194.4 mm to (50.8, 26.7), turned to 90 degrees
- moved R18 192.0 mm to (58.4, 25.4)
- moved C12 188.1 mm to (53.3, 27.9), turned to 270 degrees
- moved R15 173.6 mm to (59.7, 30.5), turned to 180 degrees
- moved R13 172.8 mm to (68.6, 34.3), turned to 270 degrees
- moved R14 170.7 mm to (66.0, 27.9), turned to 270 degrees
- moved R17 168.4 mm to (45.7, 26.7), turned to 180 degrees
- moved C10 168.1 mm to (66.0, 35.6), turned to 90 degrees
- moved C7 163.3 mm to (57.1, 67.3), turned to 270 degrees
- moved R12 162.8 mm to (54.6, 63.5), turned to 270 degrees
- moved C9 159.7 mm to (36.8, 53.3), turned to 180 degrees
- moved C8 138.5 mm to (50.8, 52.1), turned to 270 degrees
- moved R11 134.9 mm to (44.5, 48.3), turned to 90 degrees
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Connections:
- new net DATA40_1: SL1.5, U$4.1A
- new net DATA40_2: SL1.7, U$2.5, U$3.5, U$4.1B
- new net DATA40_3: SL1.9, U$2.7, U$3.7, U$4.1C
- new net DATA80_1: SL1.4, U$4.2A
- new net DATA80_2: SL1.6, U$2.4, U$3.4, U$4.2B
- new net DATA80_3: SL1.8, U$2.6, U$3.6, U$4.2C
- new net INPUT: INPUT.1, R1.1
- new net N$27: R19.1, R9.2
- new net N$28: R11.2, R20.1
- new net N$29: C16.1, R24.1, R25.2
- new net N$30: C15.2, IC2.12, R24.2
- new net N$31: C13.1, C14.2, R21.1
- new net N$32: IC2.1, IC2.2, IC2.5, JP2.1, R21.2
- new net N$33: C14.1, IC2.3, R23.1
- new net N$34: C16.2, IC2.10, IC2.13, IC2.14, JP3.1
- new net N$35: R22.2, R25.1
- new net N$36: R27.2, U$3.DEL_V_-
- new net OUT_40: IC2.7, U$4.COM_1
- new net OUT_80: IC2.8, U$4.COM_2
- net +15V: now also C17.2, C19.2, C20.2, SL1.1, U$2.1, U$2.DEL_V_+, U$3.1, U$3.DEL_V_+; no longer JP1.1
- net -15V: now also C18.1, C21.1, C22.1, SL1.2, U$2.3, U$3.3; no longer JP1.3
- net GND: now also C15.1, C17.1, C18.2, C19.1, C20.1, C21.2, C22.2, IC2.6, IC2.9, IC3.10, INPUT.2, R23.2, R26.1, R27.1, SL1.3, U$2.2, U$2.8, U$3.2, U$3.8; no longer IC3.12, JP1.2
- net N$11: now also R26.2, U$2.DEL_V_-; no longer R1.1
- net N$12: now also R19.2; no longer R9.2
- net N$16: now also R20.2; no longer R11.2
- net N$18: now also C13.2
- net N$2: now also IC3.9; no longer IC3.13
- net N$20: now also IC1.13, IC1.14; no longer IC1.8, IC1.9
- net N$21: now also IC1.12; no longer IC1.10
- net N$24: now also IC1.8, IC1.9, R22.1; no longer IC1.13, IC1.14
- net N$25: now also IC1.10; no longer IC1.12
- net N$3: now also IC3.8, JP1.1; no longer IC3.14
Routing:
- net -15V: track 0.00 -> 250.0 mm, vias 0 -> 3
- net +15V: track 0.00 -> 222.6 mm, vias 0 -> 2
- net DATA40_2: track 0.00 -> 106.5 mm, vias 0 -> 1
- net DATA40_3: track 0.00 -> 81.3 mm, vias 0 -> 1
- net N$19: track 0.00 -> 78.0 mm
- net DATA80_2: track 0.00 -> 75.4 mm, vias 0 -> 2
- net DATA80_3: track 0.00 -> 63.7 mm, vias 0 -> 2
- net OUT_40: track 0.00 -> 53.2 mm, vias 0 -> 2
- net N$17: track 0.00 -> 40.6 mm
- net N$2: track 0.00 -> 35.7 mm
- net N$27: track 0.00 -> 33.6 mm
- net N$32: track 0.00 -> 32.8 mm
- net N$3: track 0.00 -> 28.8 mm
- net OUT_80: track 0.00 -> 27.0 mm
- net N$13: track 0.00 -> 26.8 mm
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- added copper zone on layer 1, net GND
- added copper zone on layer 16, net GND
Other:
- board size 160 x 100 mm -> 72.4 x 72.4 mm

Commit message: derniere carte elec : la puissance et la communication sans fil + maj modele 3D balise receptrice
Parts:
- removed SL1: (no value), con-amp-quick:09P
- added D1: 1N4004, diode:DO41-10
- added SL2: (no value), con-amp-quick:10P
Connections:
- new net +15V_PROTECTED: C17.2, C19.2, C20.2, D1.C, IC1.4, IC2.4, IC3.4, U$1.8
- net +15V: now also D1.A, SL2.1; no longer C17.2, C19.2, C20.2, IC1.4, IC2.4, IC3.4, SL1.1, U$1.8
- net -15V: now also SL2.2; no longer SL1.2
- net DATA40_1: now also SL2.5; no longer SL1.5
- net DATA40_2: now also SL2.7; no longer SL1.7
- net DATA40_3: now also SL2.9; no longer SL1.9
- net DATA80_1: now also SL2.4; no longer SL1.4
- net DATA80_2: now also SL2.6; no longer SL1.6
- net DATA80_3: now also SL2.8; no longer SL1.8
- net GND: now also SL2.10, SL2.3; no longer SL1.3
Routing:
- net +15V: track 222.6 -> 71.4 mm, vias 2 -> 0
- net +15V_PROTECTED: track 0.00 -> 142.6 mm
- net DATA40_3: track 81.3 -> 83.8 mm, vias 1 -> 2
- net DATA40_2: track 106.5 -> 108.2 mm
- net DATA80_3: track 63.7 -> 65.3 mm
- net -15V: track 250.0 -> 251.1 mm
- net DATA80_1: track 7.55 -> 8.30 mm
- net DATA40_1: track 11.6 -> 12.3 mm
