File: electronique/balise réceptrice/balise réceptrice - puissance et communication.brd (EAGLE design)
At the start: 72.4 x 72.4 mm, 27 parts, among them IC1 786TV

Commit message: release modele 3D + elec :D
Parts:
- added LED1, LED2, LED3, LED4: (no value), led:LED3MM
- added R13: 22K, resistor:0204/7
Connections:
- new net N$23: LED1.A, U$2.6
- new net N$24: LED2.A, U$2.5
- new net N$25: LED3.A, U$2.4
- new net N$26: LED4.A, U$2.3
- new net N$27: LED1.K, LED2.K, LED3.K, LED4.K, R13.1
- net GND: now also R13.2
Routing:
- net N$27: track 0.00 -> 37.4 mm
- net N$23: track 0.00 -> 31.7 mm
- net N$24: track 0.00 -> 25.6 mm
- net N$25: track 0.00 -> 21.8 mm
- net N$26: track 0.00 -> 6.35 mm
Changed lines of the file:
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@@
 <layer number="43" name="vRestrict" color="2" fill="10" visible="yes" active="yes"/>
 <layer number="44" name="Drills" color="7" fill="1" visible="no" active="yes"/>
-<layer number="45" name="Holes" color="7" fill="1" visible="no" active="yes"/>
+<layer number="45" name="Holes" color="7" fill="1" visible="yes" active="yes"/>
 <layer number="46" name="Milling" color="3" fill="1" visible="no" active="yes"/>
 <layer number="47" name="Measures" color="7" fill="1" visible="no" active="yes"/>
@@
 <wire x1="0" y1="72.39" x2="0" y2="0" width="0" layer="20"/>
 <wire x1="0" y1="0" x2="72.39" y2="0" width="0" layer="20"/>
+<hole x="12.7" y="59.69" drill="3.2"/>
+<hole x="67.31" y="12.7" drill="3.2"/>
 </plain>
 <attributes>
@@
 <element name="DC1" library="dc-dc-converter" package="SIP3" value="R-78C5.0-1.0" x="66.04" y="58.42" rot="R180"/>
 <element name="JP1" library="jumper" package="JP1" value="" x="60.96" y="43.18" rot="R270"/>
+<element name="R13" library="resistor" package="0204/7" value="22K" x="12.7" y="8.89" rot="R270"/>
+<element name="LED1" library="led" package="LED3MM" value="" x="44.45" y="6.35" rot="R270"/>
+<element name="LED2" library="led" package="LED3MM" value="" x="36.195" y="6.35" rot="R270"/>
+<element name="LED3" library="led" package="LED3MM" value="" x="27.94" y="6.35" rot="R270"/>
+<element name="LED4" library="led" package="LED3MM" value="" x="12.7" y="16.51" rot="R270"/>
 </elements>
 <signals>
@@
 </polygon>
 <contactref element="JP1" pad="1"/>
+<contactref element="R13" pad="2"/>
 </signal>
 <signal name="-15V">
@@
 <wire x1="68.58" y1="43.18" x2="68.58" y2="58.42" width="0.8128" layer="16"/>
 </signal>
+<signal name="N$23">
+<contactref element="U$2" pad="6"/>
+<contactref element="LED1" pad="A"/>
+<wire x1="20.32" y1="24.13" x2="31.75" y2="12.7" width="0.4064" layer="16"/>
+<wire x1="31.75" y1="12.7" x2="40.64" y2="12.7" width="0.4064" layer="16"/>
+<wire x1="40.64" y1="12.7" x2="44.45" y2="8.89" width="0.4064" layer="16"/>
+<wire x1="44.45" y1="8.89" x2="44.45" y2="7.62" width="0.4064" layer="16"/>
+</signal>
+<signal name="N$24">
+<contactref element="U$2" pad="5"/>
+<contactref element="LED2" pad="A"/>
+<wire x1="17.78" y1="24.13" x2="30.48" y2="11.43" width="0.4064" layer="16"/>
+<wire x1="30.48" y1="11.43" x2="33.02" y2="11.43" width="0.4064" layer="16"/>
+<wire x1="33.02" y1="11.43" x2="36.195" y2="8.255" width="0.4064" layer="16"/>
+<wire x1="36.195" y1="8.255" x2="36.195" y2="7.62" width="0.4064" layer="16"/>
+</signal>
+<signal name="N$25">
+<contactref element="U$2" pad="4"/>
+<contactref element="LED3" pad="A"/>
+<wire x1="15.24" y1="24.13" x2="27.94" y2="11.43" width="0.4064" layer="16"/>
+<wire x1="27.94" y1="11.43" x2="27.94" y2="7.62" width="0.4064" layer="16"/>
+</signal>
+<signal name="N$26">
+<contactref element="U$2" pad="3"/>
+<contactref element="LED4" pad="A"/>
+<wire x1="12.7" y1="24.13" x2="12.7" y2="17.78" width="0.4064" layer="16"/>
+</signal>
+<signal name="N$27">
+<contactref element="LED4" pad="K"/>
+<contactref element="R13" pad="1"/>
+<contactref element="LED3" pad="K"/>
+<contactref element="LED2" pad="K"/>
+<contactref element="LED1" pad="K"/>
+<wire x1="12.7" y1="15.24" x2="12.7" y2="12.7" width="0.4064" layer="16"/>
+<wire x1="27.94" y1="5.08" x2="20.32" y2="5.08" width="0.4064" layer="16"/>
+<wire x1="20.32" y1="5.08" x2="12.7" y2="12.7" width="0.4064" layer="16"/>
+<wire x1="27.94" y1="5.08" x2="36.195" y2="5.08" width="0.4064" layer="16"/>
+<wire x1="36.195" y1="5.08" x2="44.45" y2="5.08" width="0.4064" layer="16"/>
+</signal>
 </signals>

Commit message: ajout des fichiers gerber et excellon
Parts:
- added U$3: 1RT, switch:1RT
Connections:
- new net N$28: SUPPLY.2, U$3.2
- net N$22: now also U$3.3; no longer SUPPLY.2
Routing:
- net N$28: track 0.00 -> 8.67 mm
- net N$22: track 15.2 -> 21.7 mm
- net +3V3: track 48.6 -> 47.6 mm
Changed lines of the file:
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@@
 <layer number="27" name="tValues" color="7" fill="1" visible="yes" active="yes"/>
 <layer number="28" name="bValues" color="7" fill="1" visible="yes" active="yes"/>
-<layer number="29" name="tStop" color="7" fill="3" visible="no" active="yes"/>
-<layer number="30" name="bStop" color="7" fill="6" visible="no" active="yes"/>
-<layer number="31" name="tCream" color="7" fill="4" visible="no" active="yes"/>
-<layer number="32" name="bCream" color="7" fill="5" visible="no" active="yes"/>
-<layer number="33" name="tFinish" color="6" fill="3" visible="no" active="yes"/>
-<layer number="34" name="bFinish" color="6" fill="6" visible="no" active="yes"/>
-<layer number="35" name="tGlue" color="7" fill="4" visible="no" active="yes"/>
-<layer number="36" name="bGlue" color="7" fill="5" visible="no" active="yes"/>
-<layer number="37" name="tTest" color="7" fill="1" visible="no" active="yes"/>
-<layer number="38" name="bTest" color="7" fill="1" visible="no" active="yes"/>
+<layer number="29" name="tStop" color="7" fill="3" visible="yes" active="yes"/>
+<layer number="30" name="bStop" color="7" fill="6" visible="yes" active="yes"/>
+<layer number="31" name="tCream" color="7" fill="4" visible="yes" active="yes"/>
+<layer number="32" name="bCream" color="7" fill="5" visible="yes" active="yes"/>
+<layer number="33" name="tFinish" color="6" fill="3" visible="yes" active="yes"/>
+<layer number="34" name="bFinish" color="6" fill="6" visible="yes" active="yes"/>
+<layer number="35" name="tGlue" color="7" fill="4" visible="yes" active="yes"/>
+<layer number="36" name="bGlue" color="7" fill="5" visible="yes" active="yes"/>
+<layer number="37" name="tTest" color="7" fill="1" visible="yes" active="yes"/>
+<layer number="38" name="bTest" color="7" fill="1" visible="yes" active="yes"/>
 <layer number="39" name="tKeepout" color="4" fill="11" visible="yes" active="yes"/>
 <layer number="40" name="bKeepout" color="1" fill="11" visible="yes" active="yes"/>
@@
 <layer number="42" name="bRestrict" color="1" fill="10" visible="yes" active="yes"/>
 <layer number="43" name="vRestrict" color="2" fill="10" visible="yes" active="yes"/>
-<layer number="44" name="Drills" color="7" fill="1" visible="no" active="yes"/>
+<layer number="44" name="Drills" color="7" fill="1" visible="yes" active="yes"/>
 <layer number="45" name="Holes" color="7" fill="1" visible="yes" active="yes"/>
-<layer number="46" name="Milling" color="3" fill="1" visible="no" active="yes"/>
-<layer number="47" name="Measures" color="7" fill="1" visible="no" active="yes"/>
+<layer number="46" name="Milling" color="3" fill="1" visible="yes" active="yes"/>
+<layer number="47" name="Measures" color="7" fill="1" visible="yes" active="yes"/>
 <layer number="48" name="Document" color="7" fill="1" visible="yes" active="yes"/>
 <layer number="49" name="Reference" color="7" fill="1" visible="yes" active="yes"/>
@@
 <hole x="12.7" y="59.69" drill="3.2"/>
 <hole x="67.31" y="12.7" drill="3.2"/>
+<dimension x1="0" y1="72.39" x2="0" y2="0" x3="-12.7" y3="36.195" layer="47"/>
+<dimension x1="0" y1="72.39" x2="72.39" y2="72.39" x3="36.195" y3="78.74" layer="47"/>
 </plain>
 <attributes>
@@
 <element name="LED3" library="led" package="LED3MM" value="" x="27.94" y="6.35" rot="R270"/>
 <element name="LED4" library="led" package="LED3MM" value="" x="12.7" y="16.51" rot="R270"/>
+<element name="U$3" library="switch" package="1RT" value="1RT" x="69.85" y="36.83" rot="R90"/>
 </elements>
 <signals>
@@
 <wire x1="52.07" y1="43.18" x2="55.88" y2="39.37" width="0.4064" layer="16"/>
 <wire x1="55.88" y1="39.37" x2="64.77" y2="39.37" width="0.4064" layer="16"/>
-<wire x1="64.77" y1="39.37" x2="67.31" y2="36.83" width="0.4064" layer="16"/>
-<wire x1="67.31" y1="36.83" x2="67.31" y2="20.32" width="0.4064" layer="16"/>
-<wire x1="67.31" y1="20.32" x2="64.77" y2="17.78" width="0.4064" layer="16"/>
+<wire x1="64.77" y1="39.37" x2="66.04" y2="38.1" width="0.4064" layer="16"/>
+<wire x1="66.04" y1="38.1" x2="66.04" y2="19.05" width="0.4064" layer="16"/>
+<wire x1="66.04" y1="19.05" x2="64.77" y2="17.78" width="0.4064" layer="16"/>
 <wire x1="64.77" y1="17.78" x2="64.45" y2="17.78" width="0.4064" layer="16"/>
 <wire x1="64.45" y1="17.78" x2="64.34" y2="17.67" width="0.4064" layer="16"/>
@@
 <contactref element="JP1" pad="2"/>
 <wire x1="66.04" y1="43.18" x2="62.23" y2="43.18" width="0.8128" layer="16"/>
-</signal>
-<signal name="N$22">
-<contactref element="SUPPLY" pad="2"/>
-<contactref element="DC1" pad="1"/>
-<wire x1="68.58" y1="43.18" x2="68.58" y2="58.42" width="0.8128" layer="16"/>
 </signal>
 <signal name="N$23">
@@
 <wire x1="36.195" y1="5.08" x2="44.45" y2="5.08" width="0.4064" layer="16"/>
 </signal>
+<signal name="N$22">
+<contactref element="DC1" pad="1"/>
+<contactref element="U$3" pad="3"/>
+<wire x1="68.58" y1="58.42" x2="71.755" y2="55.245" width="0.8128" layer="16"/>
+<wire x1="71.755" y1="55.245" x2="71.755" y2="40.735" width="0.8128" layer="16"/>
+<wire x1="71.755" y1="40.735" x2="69.85" y2="38.83" width="0.8128" layer="16"/>
+</signal>
+<signal name="N$28">
+<contactref element="SUPPLY" pad="2"/>
+<contactref element="U$3" pad="2"/>
+<wire x1="68.58" y1="43.18" x2="68.58" y2="41.91" width="0.8128" layer="16"/>
+<wire x1="68.58" y1="41.91" x2="67.31" y2="40.64" width="0.8128" layer="16"/>
+<wire x1="67.31" y1="40.64" x2="67.31" y2="38.1" width="0.8128" layer="16"/>
+<wire x1="67.31" y1="38.1" x2="68.58" y2="36.83" width="0.8128" layer="16"/>
+<wire x1="68.58" y1="36.83" x2="69.85" y2="36.83" width="0.8128" layer="16"/>
+</signal>
 </signals>

Commit message: Ajout doc + mise a jour des modeles 3D
Parts:
- R13: value 22K -> 220
Changed lines of the file:
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@@
 <element name="DC1" library="dc-dc-converter" package="SIP3" value="R-78C5.0-1.0" x="66.04" y="58.42" rot="R180"/>
 <element name="JP1" library="jumper" package="JP1" value="" x="60.96" y="43.18" rot="R270"/>
-<element name="R13" library="resistor" package="0204/7" value="22K" x="12.7" y="8.89" rot="R270"/>
+<element name="R13" library="resistor" package="0204/7" value="220" x="12.7" y="8.89" rot="R270"/>
 <element name="LED1" library="led" package="LED3MM" value="" x="44.45" y="6.35" rot="R270"/>
 <element name="LED2" library="led" package="LED3MM" value="" x="36.195" y="6.35" rot="R270"/>
